Commit message: rebuild

File: catkin_ws/src/car_robot_model/urdf/include/sensors.xacro (robot description, xacro)
@@ -90,12 +90,4 @@
         <origin xyz="0.035 -0.035 0.0025" rpy="0 0 0"/>
     </joint>
-    <!-- BNO055 -->
-    <link name="bno055">
-    </link>
-    <joint name="joint_sensor_board_to_bno055" type="fixed">
-        <parent link="sensor_board"/>
-        <child link="bno055"/>
-        <origin xyz="0.235 0.0 0.023" rpy="0 0 1.5708"/>
-    </joint>
     <!-- Odroid -->
     <link name="odroid">
